File: hardware/Bibi.kicad_sch (KiCad schematic)
At the start: 9 parts, among them M1 Motor_Servo, M2 Motor_Servo, M3 Fan_3pin

Commit message: add footprints
Parts:
- removed BT1: Battery, symbol Device:Battery
- J1, J2: footprint (none) -> Connector_PinHeader_2.00mm:PinHeader_1x28_P2.00mm_Vertical
- R1: value 51K -> 1.5K; footprint (none) -> Resistor_THT:R_Axial_DIN0411_L9.9mm_D3.6mm_P12.70mm_Horizontal
- R2: value 62K -> 6.8K; footprint (none) -> Resistor_THT:R_Axial_DIN0411_L9.9mm_D3.6mm_P12.70mm_Horizontal
Connections:
- net 3.3V_1 is gone; now on net 3.3V: J2.2 (Pin_2)
- net 5V_1 is gone; now on net 5V: J2.1 (Pin_1)

Commit message: pcb file started
Parts:
- added BT1: Battery, symbol Device:Battery
Connections:
- net GND: now also BT1.2 (-)
- net at R1.1: now also BT1.1 (+)
Changed lines of the file:
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@@
 (kicad_sch
-	(version 20231120)
+	(version 20250114)
 	(generator "eeschema")
-	(generator_version "8.0")
+	(generator_version "9.0")
 	(paper "A4")
+	(rectangle
+		(start 231.14 106.68)
+		(end 262.89 67.31)
+		(stroke
+			(width 0)
+			(type default)
+		)
+		(fill
+			(type none)
+		)
+	)
+	(rectangle
+		(start 25.4 76.2)
+		(end 76.2 140.97)
+		(stroke
+			(width 0)
+			(type default)
+		)
+		(fill
+			(type none)
+		)
+	)
+	(rectangle
+		(start 34.29 22.86)
+		(end 73.66 64.77)
+		(stroke
+			(width 0)
+			(type default)
+		)
+		(fill
+			(type none)
+		)
+	)
+	(rectangle
+		(start 220.98 22.86)
+		(end 273.05 60.96)
+		(stroke
+			(width 0)
+			(type default)
+		)
+		(fill
+			(type none)
+		)
+	)
+	(text "Fan (Vaccuum)\n"
+		(exclude_from_sim no)
+		(at 246.126 71.628 0)
+		(effects
+			(font
+				(size 1.27 1.27)
+			)
+		)
+	)
+	(text "Servo (Bibi Move)\n"
+		(exclude_from_sim no)
+		(at 241.554 26.924 0)
+		(effects
+			(font
+				(size 1.27 1.27)
+			)
+		)
+	)
+	(text "Power Source (Battery)\n"
+		(exclude_from_sim no)
+		(at 49.53 25.654 0)
+		(effects
+			(font
+				(size 1.27 1.27)
+			)
+		)
+	)
+	(text "PWM 10B\n"
+		(exclude_from_sim no)
+		(at 255.016 58.42 0)
+		(effects
+			(font
+				(size 1.27 1.27)
+			)
+		)
+	)
+	(text "PWM 9B\n"
+		(exclude_from_sim no)
+		(at 249.428 99.314 0)
+		(effects
+			(font
+				(size 1.27 1.27)
+			)
+		)
+	)
+	(text "TFT Screen (Bibi Face)\n"
+		(exclude_from_sim no)
+		(at 49.276 79.502 0)
+		(effects
+			(font
+				(size 1.27 1.27)
+			)
+		)
+	)
+	(text "PWM 10A\n"
+		(exclude_from_sim no)
+		(at 228.854 58.42 0)
+		(effects
+			(font
+				(size 1.27 1.27)
+			)
+		)
+	)
 	(junction
 		(at 55.88 41.91)
@@
 			(width 0)
 			(type default)
-		)
-	)
-	(rectangle
-		(start 231.14 106.68)
-		(end 262.89 67.31)
-		(stroke
-			(width 0)
-			(type default)
-		)
-		(fill
-			(type none)
-		)
-	)
-	(rectangle
-		(start 25.4 76.2)
-		(end 76.2 140.97)
-		(stroke
-			(width 0)
-			(type default)
-		)
-		(fill
-			(type none)
-		)
-	)
-	(rectangle
-		(start 34.29 22.86)
-		(end 73.66 64.77)
-		(stroke
-			(width 0)
-			(type default)
-		)
-		(fill
-			(type none)
-		)
-	)
-	(rectangle
-		(start 220.98 22.86)
-		(end 273.05 60.96)
-		(stroke
-			(width 0)
-			(type default)
-		)
-		(fill
-			(type none)
-		)
-	)
-	(text "Fan (Vaccuum)\n"
-		(exclude_from_sim no)
-		(at 246.126 71.628 0)
-		(effects
-			(font
-				(size 1.27 1.27)
-			)
-		)
-	)
-	(text "Servo (Bibi Move)\n"
-		(exclude_from_sim no)
-		(at 241.554 26.924 0)
-		(effects
-			(font
-				(size 1.27 1.27)
-			)
-		)
-	)
-	(text "Power Source (Battery)\n"
-		(exclude_from_sim no)
-		(at 49.53 25.654 0)
-		(effects
-			(font
-				(size 1.27 1.27)
-			)
-		)
-	)
-	(text "PWM 10B\n"
-		(exclude_from_sim no)
-		(at 255.016 58.42 0)
-		(effects
-			(font
-				(size 1.27 1.27)
-			)
-		)
-	)
-	(text "PWM 9B\n"
-		(exclude_from_sim no)
-		(at 249.428 99.314 0)
-		(effects
-			(font
-				(size 1.27 1.27)
-			)
-		)
-	)
-	(text "TFT Screen (Bibi Face)\n"
-		(exclude_from_sim no)
-		(at 49.276 79.502 0)
-		(effects
-			(font
-				(size 1.27 1.27)
-			)
-		)
-	)
-	(text "PWM 10A\n"
-		(exclude_from_sim no)
-		(at 228.854 58.42 0)
-		(effects
-			(font
-				(size 1.27 1.27)
-			)
 		)
 	)
@@
 	)
 	(symbol
+		(lib_id "Device:Battery")
+		(at 40.64 38.1 0)
+		(unit 1)
+		(exclude_from_sim no)
+		(in_bom yes)
+		(on_board yes)
+		(dnp no)
+		(fields_autoplaced yes)
+		(property "Reference" "BT1"
+			(at 44.45 36.2584 0)
+			(effects
+				(font
+					(size 1.27 1.27)
+				)
+				(justify left)
+			)
+		)
+		(property "Value" "Battery"
+			(at 44.45 38.7984 0)
+			(effects
+				(font
+					(size 1.27 1.27)
+				)
+				(justify left)
+			)
+		)
+		(property "Footprint" ""
+			(at 40.64 36.576 90)
+			(effects
+				(font
+					(size 1.27 1.27)
+				)
+				(hide yes)
+			)
+		)
+		(property "Datasheet" "~"
+			(at 40.64 36.576 90)
+			(effects
+				(font
+					(size 1.27 1.27)
+				)
+				(hide yes)
+			)
+		)
+		(property "Description" "Multiple-cell battery"
+			(at 40.64 38.1 0)
+			(effects
+				(font
+					(size 1.27 1.27)
+				)
+				(hide yes)
+			)
+		)
+		(pin "2"
+		)
+		(pin "1"
+		)
+		(instances
+			(project ""
+				(path "/8a2f99a2-cef3-4cf9-b8b2-3729cb06efb7"
+					(reference "BT1")
+					(unit 1)
+				)
+			)
+		)
+	)
+	(symbol
 		(lib_id "power:GND")
 		(at 40.64 48.26 0)
@@
 		)
 	)
+	(embedded_fonts no)
 )

Commit message: new wiring
Parts:
- added J3: ~, Connector_PinSocket_2.54mm:PinSocket_1x04_P2.54mm_Vertical, symbol Connector:Conn_01x04_Socket
- added J4: ~, Connector_PinSocket_2.54mm:PinSocket_1x03_P2.54mm_Vertical, symbol Connector:Conn_01x03_Socket
- added U2: Left, OptoDevice:Vishay_MOLD-3Pin, symbol Interface_Optical:TSDP341xx
- added U3: Right, OptoDevice:Everlight_IRM-H6xxT, symbol Interface_Optical:IRM-H6xxT
- added U4: GP2Y0A51SK0F, OptoDevice:Vishay_MOLD-3Pin, symbol Interface_Optical:TSDP341xx
- J1, J2: footprint Connector_PinHeader_2.00mm:PinHeader_1x28_P2.00mm_Vertical -> Connector_PinSocket_2.54mm:PinSocket_1x28_P2.54mm_Vertical
Connections:
- net 0: now also U1.4 (RESET)
- net 1: now also U1.3 (~{CS})
- net 12: no longer U1.4 (RESET)
- net 13: no longer U1.3 (~{CS})
- net 14: no longer U1.7 (SCK)
- net 15: no longer U1.6 (MOSI)
- net 17: no longer U1.5 (D/~{C})
- net 2: now also U1.7 (SCK)
- net 3: now also U1.6 (MOSI)
- net 3.3V: now also J3.1 (Pin_1)
- net 39: now also U3.3 (OUT)
- net 47: now also U4.1 (OUT)
- net 5: now also U1.5 (D/~{C})
- net 5V: now also U2.3 (Vs), U3.4 (Vcc), U4.3 (Vs)
- net 8: now also U2.1 (OUT)
- net GND: now also J3.2 (Pin_2), J4.2 (Pin_2), U2.2 (GND), U3.1 (GND), U3.2 (GND), U4.2 (GND)
Other:
- note added: "ADC Channel 7"
- note added: "Fan (Bibi Clean)"
- note added: "IR Sensors (Bibi see)"
- note added: "Power Source (Bibi Life)"
- note removed: "Fan (Vaccuum)"
- note removed: "Power Source (Battery)"
- moved on the sheet: BT1, M1, M2, M3, R1, R2

Commit message: updated schematic
Parts:
- removed BT1: Battery, symbol Device:Battery
- removed R1: 1.5K, Resistor_THT:R_Axial_DIN0411_L9.9mm_D3.6mm_P12.70mm_Horizontal, symbol Device:R
- removed R2: 6.8K, Resistor_THT:R_Axial_DIN0411_L9.9mm_D3.6mm_P12.70mm_Horizontal, symbol Device:R
- added Q1, Q2, Q5, Q7: PNP, symbol Simulation_SPICE:PNP
- added Q10, Q11, Q12, Q3, Q4, Q6, Q8, Q9: NPN, symbol Simulation_SPICE:NPN
- added R10, R3, R4, R5, R6, R7, R8, R9: 1K, symbol Device:R
- added R11, R12, R13, R14: 2.6K, symbol Device:R
Connections:
- net 0: no longer U1.4 (RESET)
- net 19: now also R13.1
- net 20: now also R11.1
- net 27: now also R12.1
- net 28: now also R14.1
- net 3.3V: now also U2.3 (Vs), U3.4 (Vcc); no longer J3.1 (Pin_1)
- net 36: no longer M1.1 (PWM)
- net 37: no longer M2.1 (PWM)
- net 39: no longer U3.3 (OUT)
- net 4: now also U1.4 (RESET)
- net 5V: now also Q10.1 (C), Q11.1 (C), Q12.1 (C), Q9.1 (C), R10.2, R3.1, R4.2, R5.1, R6.2, R7.1, R8.2, R9.1; no longer M1.2 (+), M2.2 (+), U2.3 (Vs), U3.4 (Vcc)
- net 7: now also U2.1 (OUT)
- net 8: now also U3.3 (OUT); no longer U2.1 (OUT)
- net GND: now also Q10.3 (E), Q11.3 (E), Q12.3 (E), Q3.3 (E), Q4.3 (E), Q9.3 (E); no longer M1.3 (-), M2.3 (-)
- new net: Q9.2 (B), R11.2
- new net: Q7.2 (B), R9.2
- new net: Q1.2 (B), R3.2
- new net: Q6.2 (B), R8.1
- new net: Q4.2 (B), R6.1
- new net: Q5.2 (B), R7.2
- new net: Q12.2 (B), R14.2
- new net: Q2.2 (B), R5.2
- new net: Q3.2 (B), R4.1
- new net: Q8.2 (B), R10.1
- new net: Q6.3 (E), Q8.3 (E)
- new net: Q10.2 (B), R12.2
- new net: Q11.2 (B), R13.2
- new net M1_A: M1.2 (+), Q1.1 (C), Q3.1 (C)
- new net M1_B: M1.3 (-), Q2.1 (C), Q4.1 (C)
- new net M1_PWM: M1.1 (PWM), Q1.3 (E), Q2.3 (E)
- new net M2_A: M2.2 (+), Q5.1 (C), Q6.1 (C)
- new net M2_B: M2.3 (-), Q7.1 (C), Q8.1 (C)
- new net M2_PWM: M2.1 (PWM), Q5.3 (E), Q7.3 (E)
- no-connect marks 0 -> 11
Other:
- note added: "H Bridge and other power control"
- note added: "Note: GPIO Pins can only out 3.3V In order to induce saturation the gates of the H bridge must receive 5V"
- note added: "PWM 4A"
- note added: "PWM 4B"
- note removed: "PWM 10A"
- note removed: "PWM 10B"
- note removed: "Power Source (Bibi Life)"
- moved on the sheet: J1, J2, J3, J4, M1, M3, U2, U3, U4
