File: hardware/_autosave-Bibi.kicad_sch (KiCad schematic)
At the start: 39 parts, among them M1 Motor_Servo, M2 Motor_Servo, M3 Fan_3pin, Q1 PNP, Q10 NPN, Q11 NPN, Q12 NPN, Q2 PNP, Q3 NPN, Q4 NPN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

Commit message: schema update
Connections:
- net 19: now also U2.1 (OUT)
- net 7: no longer U2.1 (OUT)
Changed lines of the file:
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@@
 		)
 	)
-	(label "7"
+	(label "19"
 		(at 224.79 127 0)
 		(effects
